Commit message: fix target210 trajectory and unhook tool pose

File: generated_urdf/irb4600_60_205_gazebo.urdf (robot description, URDF)
Before this commit: robot abb_irb4600_60_205, 11 links, 10 joints
Links:
- added link unhook_tool_link, mass 0.5; collision mesh filename=file:///home/gen/abb4600_rws_ws/src/abb4600_gazebo/models/u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 scale=0.001 0.001 0.001; visual mesh filename=file:///home/gen/abb4600_rws_ws/src/abb4600_gazebo/models/u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 scale=0.001 0.001 0.001
Joints:
- added joint tool0_to_unhook_tool: type fixed, parent tool0, child unhook_tool_link, origin xyz=0 0 0 rpy=0 0 0
